Commit message: Add files via upload

File: src/robot_description/urdf/actuator/caster.urdf.xacro (robot description, xacro)
@@ -2,42 +2,42 @@
 <robot xmlns:xacro="http://www.ros.org/wiki/xacro">
     <xacro:macro name="caster_xacro" params="caster_name xyz">
-     <!-- Gazebo 颜色管理 -->
+     <!-- gazebo 色彩管理 -->
         <gazebo reference="${caster_name}_caster_link">
-            <material>Gazebo/Grey</material> <!-- 设置 Gazebo 中的材料颜色为灰色 -->
+            <material>Gazebo/Grey</material>
         </gazebo>
     <!-- ============万向轮============ -->
-        <link name="${caster_name}_caster_link"> <!-- 定义万向轮的链接 -->
+        <link name="${caster_name}_caster_link">
             <visual>
-                <origin xyz="0 0 0" rpy="0.0 0.0 0.0"/> <!-- 视觉表示的原点和方向 -->
+                <origin xyz="0 0 0" rpy="0.0 0.0 0.0"/>
                 <geometry>
-                    <sphere radius="0.016"/> <!-- 轮子的几何形状为半径为 0.016 米的球体 -->
+                    <sphere radius="0.016"/>
                 </geometry>
-                <material name="yellow"> <!-- 定义视觉材料为黄色 -->
-                    <color rgba="1.0 1.0 0.0 0.8"/> <!-- 颜色 RGBA，黄色，80% 不透明 -->
+                <material name="yellow">
+                    <color rgba="1.0 1.0 0.0 0.8"/>
                 </material>
             </visual>
             <collision>
-                <origin xyz="0 0 0" rpy="0.0 0.0 0.0"/> <!-- 碰撞检测的原点和方向 -->
+                <origin xyz="0 0 0" rpy="0.0 0.0 0.0"/>
                 <geometry>
-                    <sphere radius="0.016"/> <!-- 碰撞几何形状同样为半径为 0.016 米的球体 -->
+                    <sphere radius="0.016"/>
                 </geometry>
-                <material name="yellow"> <!-- 定义碰撞材料为黄色 -->
-                    <color rgba="1.0 1.0 0.0 0.8"/> <!-- 颜色 RGBA，黄色，80% 不透明 -->
+                <material name="yellow">
+                    <color rgba="1.0 1.0 0.0 0.8"/>
                 </material>
             </collision>
-            <xacro:sphere_inertia m="1.0" r="0.016" /> <!-- 轮子的转动惯量，质量为 1.0 kg，半径为 0.016 米 -->
+            <xacro:sphere_inertia m="1.0" r="0.016" />
         </link>
-        <joint name="${caster_name}_caster_joint" type="fixed"> <!-- 定义固定关节 -->
-            <parent link="base_link"/> <!-- 连接到基准链接 base_link -->
-            <child link="${caster_name}_caster_link"/> <!-- 连接到万向轮链接 -->
-            <origin xyz="${xyz}"/> <!-- 设置关节的原点位置 -->
-            <axis xyz="0.0 0.0 0.0"/> <!-- 关节的轴线，这里是零向量，因为是固定关节 -->
+        <joint name="${caster_name}_caster_joint" type="fixed">
+            <parent link="base_link"/>
+            <child link="${caster_name}_caster_link"/>
+            <origin xyz="${xyz}"/>
+            <axis xyz="0.0 0.0 0.0"/>
         </joint>
-        <!-- 修改轮子的摩擦系数 -->
-        <gazebo reference="${caster_name}_caster_link">
-            <mu1 value="0.0" /> <!-- 静摩擦系数设置为 0.0 -->
-            <mu2 value="0.0" /> <!-- 动摩擦系数设置为 0.0 -->
-            <kp value="1000000000.0" /> <!-- 硬度系数设置为一个非常大的值 -->
-            <kd value="1.0" /> <!-- 阻尼系数设置为 1.0 -->
+        <!-- 修改轮子们的摩擦系数 -->
+        <gazebo reference="${caster_name}_caster_link" >
+            <mu1 value="0.0" />
+            <mu2 value="0.0" />
+            <kp value="1000000000.0" />
+            <kd value="1.0" />
         </gazebo>
     </xacro:macro>

File: src/robot_description/urdf/actuator/wheel.urdf.xacro (robot description, xacro)
@@ -2,42 +2,42 @@
 <robot xmlns:xacro="http://www.ros.org/wiki/xacro">
     <xacro:macro name="wheel_xacro" params="wheel_name xyz">
-    <!-- Gazebo 颜色管理 -->
+    <!-- gazebo 色彩管理 -->
         <gazebo reference="${wheel_name}_wheel_link">
-            <material>Gazebo/Grey</material> <!-- 设置 Gazebo 中的材料颜色为灰色 -->
+            <material>Gazebo/Grey</material>
         </gazebo>
     <!-- ==================驱动轮================ -->
-        <link name="${wheel_name}_wheel_link"> <!-- 定义驱动轮的链接 -->
+        <link name="${wheel_name}_wheel_link">
             <visual>
-                <origin xyz="0 0 0" rpy="1.57079 0 0" /> <!-- 视觉表示的原点和方向 -->
+                <origin xyz="0 0 0" rpy="1.57079 0 0" />
                 <geometry>
-                    <cylinder radius="0.032" length="0.04"/> <!-- 轮子的几何形状为半径为 0.032 米，长度为 0.04 米的圆柱 -->
+                    <cylinder radius="0.032" length="0.04"/>
                 </geometry>
-                <material name="yellow"> <!-- 定义视觉材料为黄色 -->
-                    <color rgba="1.0 1.0 0.0 0.8"/> <!-- 颜色 RGBA，黄色，80% 不透明 -->
+                <material name="yellow">
+                    <color rgba="1.0 1.0 0.0 0.8"/>
                 </material>
             </visual>
             <collision>
-                <origin xyz="0 0 0" rpy="1.57079 0 0" /> <!-- 碰撞检测的原点和方向 -->
+                <origin xyz="0 0 0" rpy="1.57079 0 0" />
                 <geometry>
-                    <cylinder radius="0.032" length="0.04"/> <!-- 碰撞几何形状同样为半径为 0.032 米，长度为 0.04 米的圆柱 -->
+                    <cylinder radius="0.032" length="0.04"/>
                 </geometry>
-                <material name="yellow"> <!-- 定义碰撞材料为黄色 -->
-                    <color rgba="1.0 1.0 0.0 0.8"/> <!-- 颜色 RGBA，黄色，80% 不透明 -->
+                <material name="yellow">
+                    <color rgba="1.0 1.0 0.0 0.8"/>
                 </material>
             </collision>
-            <xacro:cylinder_inertia m="1.0" r="0.032" h="0.04" /> <!-- 轮子的转动惯量，质量为 1.0 kg，半径为 0.032 米，长度为 0.04 米 -->
+            <xacro:cylinder_inertia m="1.0" r="0.032" h="0.04" />
         </link>
-        <joint name="${wheel_name}_wheel_joint" type="continuous"> <!-- 定义连续关节 -->
-            <parent link="base_link"/> <!-- 连接到基准链接 base_link -->
-            <child link="${wheel_name}_wheel_link"/> <!-- 连接到驱动轮链接 -->
-            <origin xyz="${xyz}"/> <!-- 设置关节的原点位置 -->
-            <axis xyz="0.0 1.0 0.0"/> <!-- 关节的旋转轴为 Y 轴 -->
+        <joint name="${wheel_name}_wheel_joint" type="continuous">
+            <parent link="base_link"/>
+            <child link="${wheel_name}_wheel_link"/>
+            <origin xyz="${xyz}"/>
+            <axis xyz="0.0 1.0 0.0"/>
         </joint>
-        <!-- 修改轮子的摩擦系数 -->
+        <!-- 修改轮子们的摩擦系数 -->
         <gazebo reference="${wheel_name}_wheel_link">
-            <mu1 value="20.0" /> <!-- 静摩擦系数设置为 20.0 -->
-            <mu2 value="20.0" /> <!-- 动摩擦系数设置为 20.0 -->
-            <kp value="1000000000.0" /> <!-- 硬度系数设置为一个非常大的值 -->
-            <kd value="1.0" /> <!-- 阻尼系数设置为 1.0 -->
+            <mu1 value="20.0" />
+            <mu2 value="20.0" />
+            <kp value="1000000000.0" />
+            <kd value="1.0" />
         </gazebo>
     </xacro:macro>

File: src/robot_description/urdf/base.urdf.xacro (robot description, xacro)
@@ -1,44 +1,40 @@
 <?xml version="1.0"?>
 <robot xmlns:xacro="http://www.ros.org/wiki/xacro">
-    <!-- 引入通用惯性参数定义的文件 -->
     <xacro:include filename="$(find robot_description)/urdf/common_inertia.xacro" />
-    <!-- 定义一个名为 base_xacro 的宏，接收 radius 和 length 两个参数 -->
     <xacro:macro name="base_xacro" params="radius length">
-        <!-- Gazebo 中的材质管理，设置基础链接的材质 -->
+        <!-- gazebo 色彩管理 -->
         <gazebo reference="base_link">
-            <material>Gazebo/CeilingTiled</material> <!-- 使用 Gazebo 内置的 CeilingTiled 材质 -->
+            <material>Gazebo/CeilingTiled</material>
         </gazebo>
-        <!-- 定义基础固定点 link，作为机器人在环境中的位置参考 -->
+        <!-- 基础固定点，可以视为机器人在环境中的位置参考 -->
         <link name="base_footprint" />
-        <!-- 创建一个固定关节，将基础固定点连接到机器人主体 -->
+        <!-- 将基础固定点连接到机器人主体 -->
         <joint name="base_joint" type="fixed">
-            <parent link="base_footprint"/> <!-- 父链接为 base_footprint -->
-            <child link="base_link"/> <!-- 子链接为 base_link -->
-            <!-- 设置关节的原点位置，xyz 表示位置，rpy 表示滚转、俯仰和偏航角 -->
+            <parent link="base_footprint"/>
+            <child link="base_link"/>
             <origin xyz="0.0 0.0 ${length/2.0+0.032-0.001}" rpy="0.0 0.0 0.0"/>
         </joint>
-        <!-- 定义机器人主体链接 base_link -->
+        <!-- 机器人主体链接 -->
         <link name="base_link">
-            <visual> <!-- 可视化表示 -->
-                <origin xyz="0 0 0.0" rpy="0 0 0" /> <!-- 设置可视化的原点位置 -->
-                <geometry> <!-- 几何形状 -->
-                    <cylinder radius="${radius}" length="${length}"/> <!-- 定义一个圆柱体，半径和长度为参数 -->
+            <visual>
+                <origin xyz="0 0 0.0" rpy="0 0 0" />
+                <geometry>
+                    <cylinder radius="${radius}" length="${length}"/>
                 </geometry>
-                <material name="white"> <!-- 设置材质为白色 -->
-                    <color rgba="1.0 1.0 1.0 0.5"/> <!-- RGBA 颜色，白色且透明度为 0.5 -->
+                <material name="white">
+                    <color rgba="1.0 1.0 1.0 0.5"/>
                 </material>
             </visual>
-            <collision> <!-- 碰撞表示 -->
-                <origin xyz="0 0 0.0" rpy="0 0 0" /> <!-- 设置碰撞的原点位置 -->
-                <geometry> <!-- 碰撞几何形状 -->
-                    <cylinder radius="${radius}" length="${length}"/> <!-- 同样定义圆柱体 -->
+            <collision>
+                <origin xyz="0 0 0.0" rpy="0 0 0" />
+                <geometry>
+                    <cylinder radius="${radius}" length="${length}"/>
                 </geometry>
-                <material name="white"> <!-- 碰撞材质为白色 -->
-                    <color rgba="1.0 1.0 1.0 0.5"/> <!-- RGBA 颜色，白色且透明度为 0.5 -->
+                <material name="white">
+                    <color rgba="1.0 1.0 1.0 0.5"/>
                 </material>
             </collision>
-            <!-- 计算圆柱体的惯性 -->
             <xacro:cylinder_inertia m="1.0" r="${radius}" h="${length}" />
         </link>
-    </xacro:macro> <!-- 宏定义结束 -->
+    </xacro:macro>
 </robot>

File: src/robot_description/urdf/common_inertia.xacro (robot description, xacro)
@@ -1,44 +1,20 @@
 <?xml version="1.0"?>
 <robot xmlns:xacro="http://www.ros.org/wiki/xacro">
-    <!-- 定义一个名为 box_inertia 的宏，用于计算长方体的惯性 -->
     <xacro:macro name="box_inertia" params="m w h d">
         <inertial>
-            <mass value="${m}"/> <!-- 设置物体的质量 -->
-            <inertia
-                ixx="${(m/12)*(h*h+d*d)}"  <!-- 绕 x 轴的惯性矩 -->
-                ixy="0.0"                  <!-- xy 平面内的惯性耦合项 -->
-                ixz="0.0"                  <!-- xz 平面内的惯性耦合项 -->
-                iyy="${(m/12)*(w*w+d*d)}"  <!-- 绕 y 轴的惯性矩 -->
-                iyz="0.0"                  <!-- yz 平面内的惯性耦合项 -->
-                izz="${(m/12)*(w*w+h*h)}"  <!-- 绕 z 轴的惯性矩 -->
-            />
+            <mass value="${m}"/>
+            <inertia ixx="${(m/12)*(h*h+d*d)}" ixy="0.0" ixz="0.0" iyy="${(m/12)*(w*w+d*d)}" iyz="0.0" izz="${(m/12)*(w*w+h*h)}" />
         </inertial>
     </xacro:macro>
-    <!-- 定义一个名为 cylinder_inertia 的宏，用于计算圆柱体的惯性 -->
     <xacro:macro name="cylinder_inertia" params="m r h">
         <inertial>
-            <mass value="${m}"/> <!-- 设置物体的质量 -->
-            <inertia
-                ixx="${(m/12)*(3*r*r+h*h)}"  <!-- 绕 x 轴的惯性矩 -->
-                ixy="0.0"                     <!-- xy 平面内的惯性耦合项 -->
-                ixz="0.0"                     <!-- xz 平面内的惯性耦合项 -->
-                iyy="${(m/12)*(3*r*r+h*h)}"  <!-- 绕 y 轴的惯性矩 -->
-                iyz="0.0"                     <!-- yz 平面内的惯性耦合项 -->
-                izz="${(m/2)*(r*r)}"          <!-- 绕 z 轴的惯性矩 -->
-            />
+            <mass value="${m}"/>
+            <inertia ixx="${(m/12)*(3*r*r+h*h)}" ixy="0.0" ixz="0.0" iyy="${(m/12)*(3*r*r+h*h)}" iyz="0.0" izz="${(m/2)*(r*r)}" />
         </inertial>
     </xacro:macro>
-    <!-- 定义一个名为 sphere_inertia 的宏，用于计算球体的惯性 -->
     <xacro:macro name="sphere_inertia" params="m r">
         <inertial>
-            <mass value="${m}"/> <!-- 设置物体的质量 -->
-            <inertia
-                ixx="${(2/5)*m*(r*r)}"  <!-- 绕 x 轴的惯性矩 -->
-                ixy="0.0"               <!-- xy 平面内的惯性耦合项 -->
-                ixz="0.0"               <!-- xz 平面内的惯性耦合项 -->
-                iyy="${(2/5)*m*(r*r)}"  <!-- 绕 y 轴的惯性矩 -->
-                iyz="0.0"               <!-- yz 平面内的惯性耦合项 -->
-                izz="${(2/5)*m*(r*r)}"  <!-- 绕 z 轴的惯性矩 -->
-            />
+            <mass value="${m}"/>
+            <inertia ixx="${(2/5)*m*(r*r)}" ixy="0.0" ixz="0.0" iyy="${(2/5)*m*(r*r)}" iyz="0.0" izz="${(2/5)*m*(r*r)}" />
         </inertial>
     </xacro:macro>

File: src/robot_description/urdf/plugins/gazebo_control_plugin.xacro (robot description, xacro)
@@ -1,28 +1,28 @@
 <?xml version="1.0"?>
 <robot xmlns:xacro="http://www.ros.org/wiki/xacro">
-    <xacro:macro name="gazebo_control_plugin"> <!-- 定义一个名为 gazebo_control_plugin 的宏 -->
+    <xacro:macro name="gazebo_control_plugin">
         <gazebo>
-            <plugin name='diff_drive' filename='libgazebo_ros_diff_drive.so'> <!-- 引入差速驱动插件 -->
+            <plugin name='diff_drive' filename='libgazebo_ros_diff_drive.so'>
                 <ros>
-                    <namespace>/</namespace> <!-- 设置 ROS 命名空间为根 -->
-                    <remapping>cmd_vel:=cmd_vel</remapping> <!-- 重映射速度命令话题 -->
-                    <remapping>odom:=odom</remapping> <!-- 重映射里程计话题 -->
+                    <namespace>/</namespace>
+                    <remapping>cmd_vel:=cmd_vel</remapping>
+                    <remapping>odom:=odom</remapping>
                 </ros>
-                <update_rate>30</update_rate> <!-- 更新速率设置为 30Hz -->
+                <update_rate>30</update_rate>
                 <!-- wheels -->
-                <left_joint>left_wheel_joint</left_joint> <!-- 左轮子关节的名称 -->
-                <right_joint>right_wheel_joint</right_joint> <!-- 右轮子关节的名称 -->
+                <left_joint>left_wheel_joint</left_joint>
+                <right_joint>right_wheel_joint</right_joint>
                 <!-- kinematics -->
-                <wheel_separation>0.2</wheel_separation> <!-- 左右轮子之间的距离（米） -->
-                <wheel_diameter>0.064</wheel_diameter> <!-- 轮子的直径（米） -->
+                <wheel_separation>0.2</wheel_separation>
+                <wheel_diameter>0.064</wheel_diameter>
                 <!-- limits -->
-                <max_wheel_torque>20</max_wheel_torque> <!-- 最大轮子扭矩（牛顿米） -->
-                <max_wheel_acceleration>1.0</max_wheel_acceleration> <!-- 最大轮子加速度（米每二次方秒） -->
+                <max_wheel_torque>20</max_wheel_torque>
+                <max_wheel_acceleration>1.0</max_wheel_acceleration>
                 <!-- output -->
-                <publish_odom>true</publish_odom> <!-- 启用里程计输出 -->
-                <publish_odom_tf>true</publish_odom_tf> <!-- 启用里程计的坐标变换输出 -->
-                <publish_wheel_tf>true</publish_wheel_tf> <!-- 启用轮子的坐标变换输出 -->
-                <odometry_frame>odom</odometry_frame> <!-- 里程计的框架名称 -->
-                <robot_base_frame>base_footprint</robot_base_frame> <!-- 机器人底部的框架名称 -->
+                <publish_odom>true</publish_odom>
+                <publish_odom_tf>true</publish_odom_tf>
+                <publish_wheel_tf>true</publish_wheel_tf>
+                <odometry_frame>odom</odometry_frame>
+                <robot_base_frame>base_footprint</robot_base_frame>
             </plugin>
         </gazebo>

File: src/robot_description/urdf/plugins/gazebo_sensor_plugin.xacro (robot description, xacro)
@@ -1,92 +1,91 @@
 <?xml version="1.0"?>
 <robot xmlns:xacro="http://www.ros.org/wiki/xacro">
-    <xacro:macro name="gazebo_sensor_plugin"> <!-- 定义一个名为 gazebo_sensor_plugin 的宏 -->
-        <!-- 激光传感器配置 -->
-        <gazebo reference="laser_link"> <!-- 关联到激光传感器的链接 -->
-            <sensor name="laserscan" type="ray"> <!-- 定义传感器类型为 ray（激光雷达） -->
-                <plugin name="laserscan" filename="libgazebo_ros_ray_sensor.so"> <!-- 加载 ROS 激光雷达插件 -->
+    <xacro:macro name="gazebo_sensor_plugin">
+        <gazebo reference="laser_link">
+            <sensor name="laserscan" type="ray">
+                <plugin name="laserscan" filename="libgazebo_ros_ray_sensor.so">
                     <ros>
-                        <namespace>/</namespace> <!-- 设置命名空间为根 -->
-                        <remapping>~/out:=scan</remapping> <!-- 重映射输出话题 -->
+                        <namespace>/</namespace>
+                        <remapping>~/out:=scan</remapping>
                     </ros>
-                    <output_type>sensor_msgs/LaserScan</output_type> <!-- 输出类型为 LaserScan 消息 -->
-                    <frame_name>laser_link</frame_name> <!-- 设置坐标框架 -->
+                    <output_type>sensor_msgs/LaserScan</output_type>
+                    <frame_name>laser_link</frame_name>
                 </plugin>
-                <always_on>true</always_on> <!-- 始终开启传感器 -->
-                <visualize>true</visualize> <!-- 可视化传感器 -->
-                <update_rate>5</update_rate> <!-- 更新频率为 5Hz -->
-                <pose>0 0 0 0 0 0</pose> <!-- 初始位姿，XYZ位置和姿态（滚转、俯仰、偏航） -->
+                <always_on>true</always_on>
+                <visualize>true</visualize>
+                <update_rate>5</update_rate>
+                <pose>0 0 0 0 0 0</pose>
+                <!-- 激光传感器配置 -->
                 <ray>
                     <!-- 设置扫描范围 -->
                     <scan>
                         <horizontal>
-                            <samples>360</samples> <!-- 扫描样本数 -->
-                            <resolution>1.000000</resolution> <!-- 分辨率 -->
-                            <min_angle>0.000000</min_angle> <!-- 最小角度 -->
-                            <max_angle>6.280000</max_angle> <!-- 最大角度（接近360度） -->
+                            <samples>360</samples>
+                            <resolution>1.000000</resolution>
+                            <min_angle>0.000000</min_angle>
+                            <max_angle>6.280000</max_angle>
                         </horizontal>
                     </scan>
                     <!-- 设置扫描距离 -->
                     <range>
-                        <min>0.120000</min> <!-- 最小检测距离 -->
-                        <max>8.0</max> <!-- 最大检测距离 -->
-                        <resolution>0.015000</resolution> <!-- 距离分辨率 -->
+                        <min>0.120000</min>
+                        <max>8.0</max>
+                        <resolution>0.015000</resolution>
                     </range>
                     <!-- 设置噪声 -->
                     <noise>
-                        <type>gaussian</type> <!-- 噪声类型为高斯噪声 -->
-                        <mean>0.0</mean> <!-- 均值 -->
-                        <stddev>0.01</stddev> <!-- 标准差 -->
+                        <type>gaussian</type>
+                        <mean>0.0</mean>
+                        <stddev>0.01</stddev>
                     </noise>
                 </ray>
             </sensor>
         </gazebo>
-        <!-- 深度相机配置 -->
-        <gazebo reference="camera_link"> <!-- 关联到相机链接 -->
-            <sensor name="camera_sensor" type="depth"> <!-- 定义传感器类型为深度相机 -->
-                <plugin name="depth_camera" filename="libgazebo_ros_camera.so"> <!-- 加载 ROS 相机插件 -->
-                    <frame_name>camera_optical_link</frame_name> <!-- 设置坐标框架 -->
+        <!-- 深度传感器 -->
+        <gazebo reference="camera_link">
+            <sensor name="camera_sensor" type="depth">
+                <plugin name="depth_camera" filename="libgazebo_ros_camera.so">
+                    <frame_name>camera_optical_link</frame_name>
                 </plugin>
-                <always_on>true</always_on> <!-- 始终开启相机 -->
-                <update_rate>10</update_rate> <!-- 更新频率为 10Hz -->
+                <always_on>true</always_on>
+                <update_rate>10</update_rate>
                 <camera name="camera">
-                    <horizontal_fov>1.5009831567</horizontal_fov> <!-- 水平视场角 -->
+                    <horizontal_fov>1.5009831567</horizontal_fov>
                     <image>
-                        <width>800</width> <!-- 图像宽度 -->
-                        <height>600</height> <!-- 图像高度 -->
-                        <format>R8G8B8</format> <!-- 图像格式 -->
+                        <width>800</width>
+                        <height>600</height>
+                        <format>R8G8B8</format>
                     </image>
-                    <distortion> <!-- 畸变参数 -->
-                        <k1>0.0</k1> <!-- 畸变参数 k1 -->
-                        <k2>0.0</k2> <!-- 畸变参数 k2 -->
-                        <k3>0.0</k3> <!-- 畸变参数 k3 -->
-                        <p1>0.0</p1> <!-- 畸变参数 p1 -->
-                        <p2>0.0</p2> <!-- 畸变参数 p2 -->
-                        <center>0.5 0.5</center> <!-- 畸变中心点 -->
+                    <distortion>
+                        <k1>0.0</k1>
+                        <k2>0.0</k2>
+                        <k3>0.0</k3>
+                        <p1>0.0</p1>
+                        <p2>0.0</p2>
+                        <center>0.5 0.5</center>
                     </distortion>
                 </camera>
             </sensor>
         </gazebo>
-        <!-- IMU传感器配置 -->
-        <gazebo reference="imu_link"> <!-- 关联到 IMU 链接 -->
-            <sensor name="imu_sensor" type="imu"> <!-- 定义传感器类型为 IMU -->
-                <plugin name="imu_plugin" filename="libgazebo_ros_imu_sensor.so"> <!-- 加载 ROS IMU 插件 -->
+        <gazebo reference="imu_link">
+            <sensor name="imu_sensor" type="imu">
+                <plugin name="imu_plugin" filename="libgazebo_ros_imu_sensor.so">
                     <ros>
-                        <namespace>/</namespace> <!-- 设置命名空间为根 -->
-                        <remapping>~/out:=imu</remapping> <!-- 重映射输出话题 -->
+                        <namespace>/</namespace>
+                        <remapping>~/out:=imu</remapping>
                     </ros>
-                    <initial_orientation_as_reference>false</initial_orientation_as_reference> <!-- 不使用初始方向作为参考 -->
+                    <initial_orientation_as_reference>false</initial_orientation_as_reference>
                 </plugin>
-                <always_on>true</always_on> <!-- 始终开启 IMU -->
-                <update_rate>100</update_rate> <!-- 更新频率为 100Hz -->
+                <always_on>true</always_on>
+                <update_rate>100</update_rate>
                 <!-- 六轴噪声设置 -->
                 <imu>
                     <angular_velocity>
                         <x>
-                            <noise type="gaussian"> <!-- 高斯噪声设置 -->
-                                <mean>0.0</mean> <!-- 均值 -->
-                                <stddev>2e-4</stddev> <!-- 标准差 -->
-                                <bias_mean>0.0000075</bias_mean> <!-- 偏差均值 -->
-                                <bias_stddev>0.0000008</bias_stddev> <!-- 偏差标准差 -->
+                            <noise type="gaussian">
+                                <mean>0.0</mean>
+                                <stddev>2e-4</stddev>
+                                <bias_mean>0.0000075</bias_mean>
+                                <bias_stddev>0.0000008</bias_stddev>
                             </noise>
                         </x>
