Commit message: Add files via upload

File: src/robot_description/urdf/robot.ros2_control.xacro (robot description, xacro)
@@ -1,50 +1,44 @@
 <?xml version="1.0"?>
 <robot xmlns:xacro="http://www.ros.org/wiki/xacro">
-    <!-- 定义一个名为 robot_ros2_control 的宏，用于设置 ROS 2 控制系统 -->
     <xacro:macro name="robot_ros2_control">
         <ros2_control name="robotGazeboSystem" type="system">
             <hardware>
-                <!-- 指定用于 ROS 2 控制的 Gazebo 系统插件 -->
                 <plugin>gazebo_ros2_control/GazeboSystem</plugin>
             </hardware>
-            <!-- 配置左轮的关节控制 -->
             <joint name="left_wheel_joint">
-                <command_interface name="velocity"> <!-- 速度控制接口 -->
-                    <param name="min">-1</param>      <!-- 最小速度 -->
-                    <param name="max">1</param>       <!-- 最大速度 -->
+                <command_interface name="velocity">
+                    <param name="min">-1</param>
+                    <param name="max">1</param>
                 </command_interface>
-                <command_interface name="effort">  <!-- 努力控制接口 -->
-                    <param name="min">-0.1</param>     <!-- 最小努力值 -->
-                    <param name="max">0.1</param>      <!-- 最大努力值 -->
+                <command_interface name="effort">
+                    <param name="min">-0.1</param>
+                    <param name="max">0.1</param>
                 </command_interface>
-                <state_interface name="position" />  <!-- 位置状态接口 -->
-                <state_interface name="velocity" />  <!-- 速度状态接口 -->
-                <state_interface name="effort" />    <!-- 努力状态接口 -->
+                <state_interface name="position" />
+                <state_interface name="velocity" />
+                <state_interface name="effort" />
             </joint>
-            <!-- 配置右轮的关节控制 -->
             <joint name="right_wheel_joint">
-                <command_interface name="velocity"> <!-- 速度控制接口 -->
-                    <param name="min">-1</param>      <!-- 最小速度 -->
-                    <param name="max">1</param>       <!-- 最大速度 -->
+                <command_interface name="velocity">
+                    <param name="min">-1</param>
+                    <param name="max">1</param>
                 </command_interface>
-                <command_interface name="effort">  <!-- 努力控制接口 -->
-                    <param name="min">-0.1</param>     <!-- 最小努力值 -->
-                    <param name="max">0.1</param>      <!-- 最大努力值 -->
+                <command_interface name="effort">
+                    <param name="min">-0.1</param>
+                    <param name="max">0.1</param>
                 </command_interface>
-                <state_interface name="position" />  <!-- 位置状态接口 -->
-                <state_interface name="velocity" />  <!-- 速度状态接口 -->
-                <state_interface name="effort" />    <!-- 努力状态接口 -->
+                <state_interface name="position" />
+                <state_interface name="velocity" />
+                <state_interface name="effort" />
             </joint>
         </ros2_control>
         <gazebo>
-            <!-- Gazebo 插件配置 -->
             <plugin filename="libgazebo_ros2_control.so" name="gazebo_ros2_control">
-                <robot_param>robot_description</robot_param>  <!-- 机器人描述参数 -->
-                <robot_param_node>robot_state_publisher</robot_param_node> <!-- 机器人状态发布者 -->
-                <parameters>$(find robot_description)/config/robot_ros2_controller.yaml</parameters> <!-- 控制器参数文件路径 -->
+                <robot_param>robot_description</robot_param>
+                <robot_param_node>robot_state_publisher</robot_param_node>
+                <parameters>$(find robot_description)/config/robot_ros2_controller.yaml</parameters>
                 <ros>
-                    <!-- ROS 话题重映射 -->
-                    <remapping>/robot_diff_drive_controller/cmd_vel_unstamped:=/cmd_vel</remapping> <!-- 重映射命令速度话题 -->
-                    <remapping>/robot_diff_drive_controller/odom:=/odom</remapping> <!-- 重映射里程计话题 -->
+                    <remapping>/robot_diff_drive_controller/cmd_vel_unstamped:=/cmd_vel</remapping>
+                    <remapping>/robot_diff_drive_controller/odom:=/odom</remapping>
                 </ros>
             </plugin>
